Commit message: Simple version of 4wheel bot with skid steer

File: laelaps_description/urdf/laelaps.xacro (robot description, xacro)
@@ -4,27 +4,85 @@
   <!-- Constants for robot dimensions -->
   <xacro:property name="PI" value="3.1415926535897931"/>
-  <xacro:property name="body_mass" value="10"/> <!-- mass of laelaps' body -->
-  <xacro:property name="body_width" value="0.042"/>
-  <xacro:property name="body_length" value="0.035"/>
-  <xacro:property name="body_height" value="0.010"/>
+  <xacro:property name="body_mass" value="35"/> <!-- mass of laelaps' body -->
+  <xacro:property name="body_width" value="0.5"/> <!-- sizeY of body-->
+  <xacro:property name="body_length" value="1.0"/> <!-- sizeX of body -->
+  <xacro:property name="body_height" value="0.25"/> <!-- sizeZ of body -->
   <!-- Import Rviz colors -->
   <xacro:include filename="$(find laelaps_description)/urdf/materials.xacro" />
+  <xacro:include filename="$(find laelaps_description)/urdf/laelaps_wheel.xacro" />
+  <!-- BASE-FOOTPRINT -->
+  <link name="base_footprint">
+    <visual>
+        <origin xyz="0 0 0" rpy="0 0 0" />
+        <geometry>
+            <box size="0.001 0.001 0.001" />
+        </geometry>
+    </visual>
+  </link>
+  <gazebo reference="base_footprint">
+    <turnGravityOff>false</turnGravityOff>
+  </gazebo>
+  <joint name="base_footprint_joint" type="fixed">
+    <origin xyz="0 0 ${body_height/2}" rpy="0 0 0" />
+    <parent link="base_footprint"/>
+    <child link="base_link" />
+  </joint>
   <!-- Body Link -->
-  <link name="body">
+  <link name="base_link">
     <visual>
       <origin xyz="0 0 ${body_height/2}" rpy="0 0 0"/>
       <geometry>
         <box size="${body_length} ${body_width} ${body_height}"/>
+        <!-- <mesh filename="package://laelaps_description/meshes/RN-LL-303-R01_scaled_compressed.stl"/>-->
       </geometry>
       <material name="orange"/>
     </visual>
+    <collision>
+      <origin xyz="0 0 0" rpy="0 0 0"/>
+      <geometry>
+        <box size="${body_length} ${body_width} ${body_height}"/>
+      </geometry>
+    </collision>
     <inertial>
-      <origin xyz="0 0 ${body_height/2}" rpy="0 0 0"/>
+      <origin xyz="0 0 0" rpy="0 0 0"/>
       <mass value="${body_mass}"/>
       <inertia
-          ixx="${body_mass/12.0 * (body_width*body_width + body_height*body_height)}" ixy="0.0" ixz="0.0"
-          iyy="${body_mass/12.0 * (body_height*body_height + body_length*body_length)}" iyz="0.0"
-          izz="${body_mass/12.0 * (body_width*body_width + body_length*body_length)}"/>
+          ixx="${(body_mass/12.0) * (body_width*body_width + body_height*body_height)}" ixy="0.0" ixz="0.0"
+          iyy="${(body_mass/12.0) * (body_height*body_height + body_length*body_length)}" iyz="0.0"
+          izz="${(body_mass/12.0) * (body_width*body_width + body_length*body_length)}"/>
     </inertial>
   </link>
+  <gazebo reference="base_link">
+    <material>Gazebo/Yellow</material>
+    <turnGravityOff>false</turnGravityOff>
+  </gazebo>
+  <!-- Wheels -->
+  <laelaps_wheel fb="front" lr="right" parent="base_link" translateX="1" translateY="-1" flipY="-1"/>
+  <laelaps_wheel fb="front" lr="left" parent="base_link" translateX="1" translateY="1" flipY="-1"/>
+  <laelaps_wheel fb="back" lr="right" parent="base_link" translateX="-1" translateY="-1" flipY="-1"/>
+  <laelaps_wheel fb="back" lr="left" parent="base_link" translateX="-1" translateY="1" flipY="-1"/>
+  <gazebo>
+    <plugin name="skid_steer_drive_controller" filename="libgazebo_ros_skid_steer_drive.so">
+      <alwaysOn>true</alwaysOn>
+      <updateRate>100.0</updateRate>
+      <leftFrontJoint>front_left_wheel_joint</leftFrontJoint>
+      <rightFrontJoint>front_right_wheel_joint</rightFrontJoint>
+      <leftRearJoint>back_left_wheel_joint</leftRearJoint>
+      <rightRearJoint>back_right_wheel_joint</rightRearJoint>
+      <wheelSeparation>${body_width}</wheelSeparation>
+      <wheelDiameter>${2*wheel_radius}</wheelDiameter>
+      <torque>1</torque>
+      <broadcastTF>1</broadcastTF>
+      <odometryFrame>map</odometryFrame>
+      <commandTopic>cmd_vel</commandTopic>
+      <odometryTopic>odom</odometryTopic>
+      <robotBaseFrame>base_link</robotBaseFrame>
+    </plugin>
+    <plugin name="gazebo_ros_control" filename="libgazebo_ros_control.so" />
+  </gazebo>
+  <gazebo>
+  <plugin name="gazebo_ros_control" filename="libgazebo_ros_control.so">
+    <robotNamespace>/laelaps</robotNamespace>
+  </plugin>
+</gazebo>
 </robot>

Commit message: Use meshes and coloring for laelaps

File: laelaps_description/urdf/laelaps.xacro (robot description, xacro)
@@ -5,9 +5,10 @@
   <xacro:property name="PI" value="3.1415926535897931"/>
   <xacro:property name="body_mass" value="35"/> <!-- mass of laelaps' body -->
-  <xacro:property name="body_width" value="0.5"/> <!-- sizeY of body-->
-  <xacro:property name="body_length" value="1.0"/> <!-- sizeX of body -->
-  <xacro:property name="body_height" value="0.25"/> <!-- sizeZ of body -->
+  <xacro:property name="body_width" value="0.25"/> <!-- sizeY of body-->
+  <xacro:property name="body_length" value="0.35"/> <!-- sizeX of body -->
+  <xacro:property name="body_height" value="0.10"/> <!-- sizeZ of body -->
+  <xacro:property name="body_z_offset" value="0.09"/> <!-- body ground clearance -->
   <!-- Import Rviz colors -->
-  <xacro:include filename="$(find laelaps_description)/urdf/materials.xacro" />
+  <!-- <xacro:include filename="$(find laelaps_description)/urdf/materials.xacro" />-->
   <xacro:include filename="$(find laelaps_description)/urdf/laelaps_wheel.xacro" />
   <!-- BASE-FOOTPRINT -->
@@ -21,8 +22,9 @@
   </link>
   <gazebo reference="base_footprint">
+    <material>Gazebo/Yellow</material>
     <turnGravityOff>false</turnGravityOff>
   </gazebo>
   <joint name="base_footprint_joint" type="fixed">
-    <origin xyz="0 0 ${body_height/2}" rpy="0 0 0" />
+    <origin xyz="0 0 ${body_z_offset}" rpy="0 0 0" />
     <parent link="base_footprint"/>
     <child link="base_link" />
@@ -31,10 +33,10 @@
   <link name="base_link">
     <visual>
-      <origin xyz="0 0 ${body_height/2}" rpy="0 0 0"/>
+      <origin xyz="0 0 ${body_z_offset}" rpy="0 0 0"/>
       <geometry>
-        <box size="${body_length} ${body_width} ${body_height}"/>
-        <!-- <mesh filename="package://laelaps_description/meshes/RN-LL-303-R01_scaled_compressed.stl"/>-->
+        <!-- <box size="${body_length} ${body_width} ${body_height}"/>-->
+        <mesh filename="package://laelaps_description/meshes/RN-LL-303-R01_scaled.stl"/>
       </geometry>
-      <material name="orange"/>
+      <material name="DarkGrey"/>
     </visual>
     <collision>
@@ -54,11 +56,10 @@
   </link>
   <gazebo reference="base_link">
-    <material>Gazebo/Yellow</material>
-    <turnGravityOff>false</turnGravityOff>
+    <material>Gazebo/DarkGrey</material>
   </gazebo>
   <!-- Wheels -->
-  <laelaps_wheel fb="front" lr="right" parent="base_link" translateX="1" translateY="-1" flipY="-1"/>
+  <laelaps_wheel fb="front" lr="right" parent="base_link" translateX="1" translateY="-1" flipY="1"/>
   <laelaps_wheel fb="front" lr="left" parent="base_link" translateX="1" translateY="1" flipY="-1"/>
-  <laelaps_wheel fb="back" lr="right" parent="base_link" translateX="-1" translateY="-1" flipY="-1"/>
+  <laelaps_wheel fb="back" lr="right" parent="base_link" translateX="-1" translateY="-1" flipY="1"/>
   <laelaps_wheel fb="back" lr="left" parent="base_link" translateX="-1" translateY="1" flipY="-1"/>
   <gazebo>
@@ -79,10 +80,10 @@
       <robotBaseFrame>base_link</robotBaseFrame>
     </plugin>
-    <plugin name="gazebo_ros_control" filename="libgazebo_ros_control.so" />
+    <!-- <plugin name="gazebo_ros_control" filename="libgazebo_ros_control.so" />-->
   </gazebo>
   <gazebo>
-  <plugin name="gazebo_ros_control" filename="libgazebo_ros_control.so">
-    <robotNamespace>/laelaps</robotNamespace>
-  </plugin>
-</gazebo>
+    <plugin name="gazebo_ros_control" filename="libgazebo_ros_control.so">
+      <robotNamespace>/laelaps</robotNamespace>
+    </plugin>
+  </gazebo>
 </robot>

File: laelaps_description/urdf/laelaps_wheel.xacro (robot description, xacro)
@@ -3,11 +3,11 @@
 <robot name="laelaps_wheel" xmlns:xacro="http://www.ros.org/wiki/xacro">
   <!-- Constants for robot dimensions -->
-  <xacro:property name="wheel_radius" value="0.2"/>
-  <xacro:property name="wheel_height" value="0.1"/>
+  <xacro:property name="wheel_radius" value="0.055"/>
+  <xacro:property name="wheel_height" value="0.06"/>
   <xacro:property name="wheel_mass" value="2.5"/>
-  <xacro:property name="base_x_origin_to_wheel_origin" value="0.25"/>
-  <xacro:property name="base_x_origin_to_wheel_origin_offset" value="0.0"/>
-  <xacro:property name="base_y_origin_to_wheel_origin" value="0.3"/>
-  <xacro:property name="base_z_origin_to_wheel_origin" value="0.0"/>
+  <xacro:property name="base_x_origin_to_wheel_origin" value="0.10"/>
+  <xacro:property name="base_x_origin_to_wheel_origin_offset" value="-0.015"/>
+  <xacro:property name="base_y_origin_to_wheel_origin" value="0.16"/>
+  <xacro:property name="base_z_origin_to_wheel_origin" value="0.00"/>
   <xacro:macro name="cylinder_inertia" params="m r h">
     <inertia ixx="${m*(3*r*r+h*h)/12}" ixy="0" ixz="0"
@@ -20,6 +20,6 @@
         <origin xyz="0 0 0" rpy="${flipY*PI/2} 0 0"/>
         <geometry>
-          <!-- <mesh filename="package://laelaps_description/meshes/wheel_scaled.stl"/> -->
-          <cylinder length="${wheel_height}" radius="${wheel_radius}"/>
+          <mesh filename="package://laelaps_description/meshes/wheel_with_rim.stl"/>
+          <!-- <cylinder length="${wheel_height}" radius="${wheel_radius}"/> -->
         </geometry>
         <material name="DarkGray"/>
@@ -43,5 +43,5 @@
       <kd  value="1.0" />
       <fdir1 value="1 0 0"/>
-      <material>Gazebo/Grey</material>
+      <material>Gazebo/DarkGrey</material>
       <turnGravityOff>false</turnGravityOff>
     </gazebo>

Commit message: Add camera and laser

File: laelaps_description/urdf/laelaps.xacro (robot description, xacro)
@@ -9,4 +9,5 @@
   <xacro:property name="body_height" value="0.10"/> <!-- sizeZ of body -->
   <xacro:property name="body_z_offset" value="0.09"/> <!-- body ground clearance -->
+  <xacro:property name="camera_link" value="0.02"/> <!-- camera box size -->
   <!-- Import Rviz colors -->
   <!-- <xacro:include filename="$(find laelaps_description)/urdf/materials.xacro" />-->
@@ -63,4 +64,126 @@
   <laelaps_wheel fb="back" lr="right" parent="base_link" translateX="-1" translateY="-1" flipY="1"/>
   <laelaps_wheel fb="back" lr="left" parent="base_link" translateX="-1" translateY="1" flipY="-1"/>
+  <joint name="camera_joint" type="fixed">
+    <axis xyz="0 1 0"/>
+    <origin xyz="${body_length/2-camera_link} 0 ${body_height-camera_link}" rpy="0 0 0"/>
+    <parent link="base_link"/>
+    <child link="camera_link"/>
+  </joint>
+  <link name="camera_link">
+    <collision>
+      <origin xyz="0 0 0" rpy="0 0 0"/>
+      <geometry>
+        <box size="0.001 0.001 0.001"/>
+      </geometry>
+    </collision>
+    <visual>
+      <origin xyz="0 0 0" rpy="0 0 0"/>
+      <geometry>
+        <box size="0.001 0.001 0.001"/>
+      </geometry>
+      <material name="red"/>
+    </visual>
+    <inertial>
+      <mass value="1e-5" />
+      <origin xyz="0 0 0" rpy="0 0 0"/>
+      <inertia ixx="1e-6" ixy="0" ixz="0" iyy="1e-6" iyz="0" izz="1e-6" />
+    </inertial>
+  </link>
+  <gazebo reference="camera_link">
+    <sensor type="camera" name="laelaps_camera">
+      <update_rate>20.0</update_rate>
+      <camera name="head">
+        <horizontal_fov>1.3962634</horizontal_fov>
+        <image>
+          <width>800</width>
+          <height>800</height>
+          <format>R8G8B8</format>
+        </image>
+        <clip>
+          <near>0.02</near>
+          <far>300</far>
+        </clip>
+        <noise>
+          <type>gaussian</type>
+          <!-- Noise is sampled independently per pixel on each frame.
+               That pixel's noise value is added to each of its color
+               channels, which at that point lie in the range [0,1]. -->
+          <mean>0.0</mean>
+          <stddev>0.007</stddev>
+        </noise>
+      </camera>
+      <plugin name="camera_controller" filename="libgazebo_ros_camera.so">
+        <alwaysOn>true</alwaysOn>
+        <updateRate>0.0</updateRate>
+        <cameraName>laelaps/laelaps_camera</cameraName>
+        <imageTopicName>image_raw</imageTopicName>
+        <cameraInfoTopicName>camera_info</cameraInfoTopicName>
+        <frameName>camera_link</frameName>
+        <hackBaseline>0.07</hackBaseline>
+        <distortionK1>0.0</distortionK1>
+        <distortionK2>0.0</distortionK2>
+        <distortionK3>0.0</distortionK3>
+        <distortionT1>0.0</distortionT1>
+        <distortionT2>0.0</distortionT2>
+      </plugin>
+    </sensor>
+  </gazebo>
+  <joint name="hokuyo_joint" type="fixed">
+    <axis xyz="0 1 0"/>
+    <origin xyz="${body_length/2} 0 ${body_height/2}" rpy="0 0 0"/>
+    <parent link="base_link"/>
+    <child link="hokuyo_link"/>
+  </joint>
+  <!--Hokuyo laser -->
+  <link name="hokuyo_link">
+    <collision>
+      <origin xyz="0 0 0" rpy="0 0 0"/>
+      <geometry>
+        <box size="0.001 0.001 0.001"/>
+      </geometry>
+    </collision>
+    <visual>
+      <origin xyz="0 0 0" rpy="0 0 0"/>
+      <geometry>
+        <box size="0.001 0.001 0.001"/>
+      </geometry>
+    </visual>
+    <inertial>
+      <mass value="1e-5"/>
+      <origin xyz="0 0 0" rpy="0 0 0"/>
+      <inertia ixx="1e-6" ixy="0" ixz="0" iyy="1e-6" iyz="0" izz="1e-6"/>
+    </inertial>
+  </link>
+  <gazebo reference="hokuyo_link">
+    <sensor type="ray" name="head_hokuyo_sensor">
+      <pose>0 0 0 0 0 0</pose>
+      <visualize>true</visualize>
+      <update_rate>20</update_rate>
+      <ray>
+        <scan>
+          <horizontal>
+            <samples>720</samples>
+            <resolution>1</resolution>
+            <min_angle>-0.2618</min_angle>
+            <max_angle>0.2618</max_angle>
+          </horizontal>
+        </scan>
+        <range>
+          <min>0.05</min>
+          <max>0.20</max>
+          <resolution>0.01</resolution>
+        </range>
+        <noise>
+          <type>gaussian</type>
+          <mean>0.0</mean>
+          <stddev>0.01</stddev>
+        </noise>
+      </ray>
+      <plugin name="gazebo_ros_head_hokuyo_controller" filename="libgazebo_ros_laser.so">
+        <topicName>/laelaps/laser/scan</topicName>
+        <frameName>hokuyo_link</frameName>
+      </plugin>
+    </sensor>
+  </gazebo>
   <gazebo>
     <plugin name="skid_steer_drive_controller" filename="libgazebo_ros_skid_steer_drive.so">
@@ -80,5 +203,4 @@
       <robotBaseFrame>base_link</robotBaseFrame>
     </plugin>
-    <!-- <plugin name="gazebo_ros_control" filename="libgazebo_ros_control.so" />-->
   </gazebo>
   <gazebo>

Commit message: Create laser macro and add three lasers

File: laelaps_description/urdf/laelaps.xacro (robot description, xacro)
@@ -10,7 +10,10 @@
   <xacro:property name="body_z_offset" value="0.09"/> <!-- body ground clearance -->
   <xacro:property name="camera_link" value="0.02"/> <!-- camera box size -->
+  <xacro:property name="laser_y_offset" value="0.063"/> <!-- distance from centerline to laser-->
+  <xacro:property name="laser_yaw" value="${15*(PI/180)}"/>
   <!-- Import Rviz colors -->
   <!-- <xacro:include filename="$(find laelaps_description)/urdf/materials.xacro" />-->
   <xacro:include filename="$(find laelaps_description)/urdf/laelaps_wheel.xacro" />
+  <xacro:include filename="$(find laelaps_description)/urdf/laelaps_laser.xacro" />
   <!-- BASE-FOOTPRINT -->
   <link name="base_footprint">
@@ -129,61 +132,8 @@
     </sensor>
   </gazebo>
-  <joint name="hokuyo_joint" type="fixed">
-    <axis xyz="0 1 0"/>
-    <origin xyz="${body_length/2} 0 ${body_height/2}" rpy="0 0 0"/>
-    <parent link="base_link"/>
-    <child link="hokuyo_link"/>
-  </joint>
-  <!--Hokuyo laser -->
-  <link name="hokuyo_link">
-    <collision>
-      <origin xyz="0 0 0" rpy="0 0 0"/>
-      <geometry>
-        <box size="0.001 0.001 0.001"/>
-      </geometry>
-    </collision>
-    <visual>
-      <origin xyz="0 0 0" rpy="0 0 0"/>
-      <geometry>
-        <box size="0.001 0.001 0.001"/>
-      </geometry>
-    </visual>
-    <inertial>
-      <mass value="1e-5"/>
-      <origin xyz="0 0 0" rpy="0 0 0"/>
-      <inertia ixx="1e-6" ixy="0" ixz="0" iyy="1e-6" iyz="0" izz="1e-6"/>
-    </inertial>
-  </link>
-  <gazebo reference="hokuyo_link">
-    <sensor type="ray" name="head_hokuyo_sensor">
-      <pose>0 0 0 0 0 0</pose>
-      <visualize>true</visualize>
-      <update_rate>20</update_rate>
-      <ray>
-        <scan>
-          <horizontal>
-            <samples>720</samples>
-            <resolution>1</resolution>
-            <min_angle>-0.2618</min_angle>
-            <max_angle>0.2618</max_angle>
-          </horizontal>
-        </scan>
-        <range>
-          <min>0.05</min>
-          <max>0.20</max>
-          <resolution>0.01</resolution>
-        </range>
-        <noise>
-          <type>gaussian</type>
-          <mean>0.0</mean>
-          <stddev>0.01</stddev>
-        </noise>
-      </ray>
-      <plugin name="gazebo_ros_head_hokuyo_controller" filename="libgazebo_ros_laser.so">
-        <topicName>/laelaps/laser/scan</topicName>
-        <frameName>hokuyo_link</frameName>
-      </plugin>
-    </sensor>
-  </gazebo>
+  <!-- Lasers -->
+  <laelaps_laser index="0" parent="base_link" translateX="${body_length/2}" translateY="0" translateZ="${body_height/2}" yaw="0"/>
+  <laelaps_laser index="1" parent="base_link" translateX="${body_length/2}" translateY="-${laser_y_offset}" translateZ="${body_height/2}" yaw="-${laser_yaw}"/>
+  <laelaps_laser index="7" parent="base_link" translateX="${body_length/2}" translateY="${laser_y_offset}" translateZ="${body_height/2}" yaw="${laser_yaw}"/>
   <gazebo>
     <plugin name="skid_steer_drive_controller" filename="libgazebo_ros_skid_steer_drive.so">

Commit message: Move camera out to macro

File: laelaps_description/urdf/laelaps.xacro (robot description, xacro)
@@ -16,4 +16,5 @@
   <xacro:include filename="$(find laelaps_description)/urdf/laelaps_wheel.xacro" />
   <xacro:include filename="$(find laelaps_description)/urdf/laelaps_laser.xacro" />
+  <xacro:include filename="$(find laelaps_description)/urdf/laelaps_camera.xacro" />
   <!-- BASE-FOOTPRINT -->
   <link name="base_footprint">
@@ -67,73 +68,11 @@
   <laelaps_wheel fb="back" lr="right" parent="base_link" translateX="-1" translateY="-1" flipY="1"/>
   <laelaps_wheel fb="back" lr="left" parent="base_link" translateX="-1" translateY="1" flipY="-1"/>
-  <joint name="camera_joint" type="fixed">
-    <axis xyz="0 1 0"/>
-    <origin xyz="${body_length/2-camera_link} 0 ${body_height-camera_link}" rpy="0 0 0"/>
-    <parent link="base_link"/>
-    <child link="camera_link"/>
-  </joint>
-  <link name="camera_link">
-    <collision>
-      <origin xyz="0 0 0" rpy="0 0 0"/>
-      <geometry>
-        <box size="0.001 0.001 0.001"/>
-      </geometry>
-    </collision>
-    <visual>
-      <origin xyz="0 0 0" rpy="0 0 0"/>
-      <geometry>
-        <box size="0.001 0.001 0.001"/>
-      </geometry>
-      <material name="red"/>
-    </visual>
-    <inertial>
-      <mass value="1e-5" />
-      <origin xyz="0 0 0" rpy="0 0 0"/>
-      <inertia ixx="1e-6" ixy="0" ixz="0" iyy="1e-6" iyz="0" izz="1e-6" />
-    </inertial>
-  </link>
-  <gazebo reference="camera_link">
-    <sensor type="camera" name="laelaps_camera">
-      <update_rate>20.0</update_rate>
-      <camera name="head">
-        <horizontal_fov>1.3962634</horizontal_fov>
-        <image>
-          <width>800</width>
-          <height>800</height>
-          <format>R8G8B8</format>
-        </image>
-        <clip>
-          <near>0.02</near>
-          <far>300</far>
-        </clip>
-        <noise>
-          <type>gaussian</type>
-          <!-- Noise is sampled independently per pixel on each frame.
-               That pixel's noise value is added to each of its color
-               channels, which at that point lie in the range [0,1]. -->
-          <mean>0.0</mean>
-          <stddev>0.007</stddev>
-        </noise>
-      </camera>
-      <plugin name="camera_controller" filename="libgazebo_ros_camera.so">
-        <alwaysOn>true</alwaysOn>
-        <updateRate>0.0</updateRate>
-        <cameraName>laelaps/laelaps_camera</cameraName>
-        <imageTopicName>image_raw</imageTopicName>
-        <cameraInfoTopicName>camera_info</cameraInfoTopicName>
-        <frameName>camera_link</frameName>
-        <hackBaseline>0.07</hackBaseline>
-        <distortionK1>0.0</distortionK1>
-        <distortionK2>0.0</distortionK2>
-        <distortionK3>0.0</distortionK3>
-        <distortionT1>0.0</distortionT1>
-        <distortionT2>0.0</distortionT2>
-      </plugin>
-    </sensor>
-  </gazebo>
+  <!-- Cameras -->
+  <laelaps_camera index="0" parent="base_link" translateX="${body_length/2-camera_link}" translateY="0" translateZ="${body_height-camera_link}"/>
   <!-- Lasers -->
   <laelaps_laser index="0" parent="base_link" translateX="${body_length/2}" translateY="0" translateZ="${body_height/2}" yaw="0"/>
   <laelaps_laser index="1" parent="base_link" translateX="${body_length/2}" translateY="-${laser_y_offset}" translateZ="${body_height/2}" yaw="-${laser_yaw}"/>
   <laelaps_laser index="7" parent="base_link" translateX="${body_length/2}" translateY="${laser_y_offset}" translateZ="${body_height/2}" yaw="${laser_yaw}"/>
+  <!-- Drivetrain -->
   <gazebo>
     <plugin name="skid_steer_drive_controller" filename="libgazebo_ros_skid_steer_drive.so">
