Commit message: Update for Kinetic

File: laelaps_description/urdf/laelaps.xacro (robot description, xacro)
@@ -41,6 +41,6 @@
       <origin xyz="0 0 ${body_z_offset}" rpy="0 0 0"/>
       <geometry>
-        <!-- <box size="${body_length} ${body_width} ${body_height}"/>-->
-        <mesh filename="package://laelaps_description/meshes/RN-LL-303-R01_scaled.stl"/>
+        <box size="${body_length} ${body_width} ${body_height}"/>
+        <!--<mesh filename="package://laelaps_description/meshes/RN-LL-303-R01_scaled.stl"/>-->
       </geometry>
       <material name="DarkGrey"/>
@@ -80,4 +80,5 @@
   <gazebo>
     <plugin name="skid_steer_drive_controller" filename="libgazebo_ros_skid_steer_drive.so">
+      <robotNamespace>/laelaps</robotNamespace>
       <alwaysOn>true</alwaysOn>
       <updateRate>100.0</updateRate>
@@ -88,5 +89,5 @@
       <wheelSeparation>${body_width}</wheelSeparation>
       <wheelDiameter>${2*wheel_radius}</wheelDiameter>
-      <torque>1</torque>
+      <torque>100</torque>
       <broadcastTF>1</broadcastTF>
       <odometryFrame>map</odometryFrame>

File: laelaps_description/urdf/laelaps_wheel.xacro (robot description, xacro)
@@ -20,6 +20,6 @@
         <origin xyz="0 0 0" rpy="${flipY*PI/2} 0 0"/>
         <geometry>
-          <mesh filename="package://laelaps_description/meshes/wheel_with_rim.stl"/>
-          <!-- <cylinder length="${wheel_height}" radius="${wheel_radius}"/> -->
+          <!--<mesh filename="package://laelaps_description/meshes/wheel_with_rim.stl"/>-->
+          <cylinder length="${wheel_height}" radius="${wheel_radius}"/>
         </geometry>
         <material name="DarkGray"/>
@@ -58,8 +58,8 @@
       <type>transmission_interface/SimpleTransmission</type>
       <joint name="${fb}_${lr}_wheel_joint">
-        <hardwareInterface>EffortJointInterface</hardwareInterface>
+        <hardwareInterface>hardware_interface/EffortJointInterface</hardwareInterface>
       </joint>
       <actuator name="${fb}_${lr}_wheel_joint_motor">
-        <hardwareInterface>EffortJointInterface</hardwareInterface>
+        <hardwareInterface>hardware_interface/EffortJointInterface</hardwareInterface>
         <mechanicalReduction>1</mechanicalReduction>
       </actuator>

Commit message: Disable IMU, Camera, and extra lasers
Update robot namespace and topics to work with nav stack
Add gazebo world for laelaps to play in

File: laelaps_description/urdf/laelaps.xacro (robot description, xacro)
@@ -70,15 +70,15 @@
   <laelaps_wheel fb="back" lr="left" parent="base_link" translateX="-1" translateY="1" flipY="-1"/>
   <!-- Cameras -->
-  <laelaps_camera index="0" parent="base_link" translateX="${body_length/2-camera_link}" translateY="0" translateZ="${body_height-camera_link}"/>
+  <!--<laelaps_camera index="0" parent="base_link" translateX="${body_length/2-camera_link}" translateY="0" translateZ="${body_height-camera_link}"/>-->
   <!-- Lasers -->
   <laelaps_laser index="0" parent="base_link" translateX="${body_length/2}" translateY="0" translateZ="${body_height/2}" yaw="0"/>
-  <laelaps_laser index="1" parent="base_link" translateX="${body_length/2}" translateY="-${laser_y_offset}" translateZ="${body_height/2}" yaw="-${laser_yaw}"/>
-  <laelaps_laser index="7" parent="base_link" translateX="${body_length/2}" translateY="${laser_y_offset}" translateZ="${body_height/2}" yaw="${laser_yaw}"/>
+  <!--<laelaps_laser index="1" parent="base_link" translateX="${body_length/2}" translateY="-${laser_y_offset}" translateZ="${body_height/2}" yaw="-${laser_yaw}"/>
+  <laelaps_laser index="7" parent="base_link" translateX="${body_length/2}" translateY="${laser_y_offset}" translateZ="${body_height/2}" yaw="${laser_yaw}"/>-->
   <!-- IMU -->
-  <laelaps_imu index="0" parent="base_link" translateX="0" translateY="0" translateZ="0"/>
+  <!--<laelaps_imu index="0" parent="base_link" translateX="0" translateY="0" translateZ="0"/>-->
   <!-- Drivetrain -->
   <gazebo>
     <plugin name="skid_steer_drive_controller" filename="libgazebo_ros_skid_steer_drive.so">
-      <robotNamespace>/laelaps</robotNamespace>
+      <robotNamespace>/</robotNamespace>
       <alwaysOn>true</alwaysOn>
       <updateRate>100.0</updateRate>
@@ -91,13 +91,13 @@
       <torque>100</torque>
       <broadcastTF>1</broadcastTF>
-      <odometryFrame>map</odometryFrame>
+      <odometryFrame>odom</odometryFrame>
       <commandTopic>cmd_vel</commandTopic>
       <odometryTopic>odom</odometryTopic>
-      <robotBaseFrame>base_link</robotBaseFrame>
+      <robotBaseFrame>base_footprint</robotBaseFrame>
     </plugin>
   </gazebo>
   <gazebo>
     <plugin name="gazebo_ros_control" filename="libgazebo_ros_control.so">
-      <robotNamespace>/laelaps</robotNamespace>
+      <robotNamespace>/</robotNamespace>
     </plugin>
   </gazebo>

File: laelaps_description/urdf/laelaps_laser.xacro (robot description, xacro)
@@ -7,5 +7,5 @@
   <xacro:property name="fovH" value="0.5236"/> <!--30 degree view angle-->
   <xacro:property name="range_min" value="0.050"/>
-  <xacro:property name="range_max" value="0.200"/>
+  <xacro:property name="range_max" value="5.00"/>
   <xacro:macro name="laelaps_laser" params="index parent translateX translateY translateZ yaw">
     <link name="laser_${index}">
@@ -44,5 +44,5 @@
           <range>
             <min>0.05</min>
-            <max>0.20</max>
+            <max>2.0</max>
             <resolution>0.01</resolution>
           </range>
@@ -54,6 +54,6 @@
         </ray>
         <plugin name="gazebo_ros_head_hokuyo_controller" filename="libgazebo_ros_laser.so">
-          <topicName>/laelaps/laser/scan</topicName>
-          <frameName>hokuyo_link</frameName>
+          <topicName>/scan</topicName>
+          <frameName>laser_0</frameName>
         </plugin>
       </sensor>
