Commit message: Set desc param before launching publisher

File: laelaps_description/urdf/laelaps_laser.xacro (robot description, xacro)
@@ -7,5 +7,5 @@
   <xacro:property name="fovH" value="0.5236"/> <!--30 degree view angle-->
   <xacro:property name="range_min" value="0.050"/>
-  <xacro:property name="range_max" value="5.00"/>
+  <xacro:property name="range_max" value="2.00"/>
   <xacro:macro name="laelaps_laser" params="index parent translateX translateY translateZ yaw">
     <link name="laser_${index}">
